File: spacecraft-health-monitor.kicad_sch (KiCad schematic)
At the start: 7 parts, among them J1 U.FL-R-SMT-1

Commit message: added INA228 VI Monitor
Parts:
- added R1: R_Shunt, symbol Device:R_Shunt
- added U2: INA228, Package_SO:TSSOP-10_3x3mm_P0.5mm, symbol Sensor_Energy:INA228
Connections:
- net GND: now also R1.4, U2.7 (GND)
- net VDD: now also R1.1, U2.8 (Vbus)
- net MCU_v_alert: now reaches U1.11 (DIO24)
- net MCU_v_alert: now also U2.3 (~{Alert})
- net MCU_v_i2c_SDA: now reaches U1.12 (DIO3)
- net MCU_v_i2c_SDA: now also U2.4 (SDA)
- net MCU_v_i2c_SCL: now reaches U1.13 (DIO4)
- net MCU_v_i2c_SCL: now also U2.5 (SCL)
- new net: R1.2, U2.10 (Vin+)
- new net: R1.3, U2.9 (Vin-)
Other:
- note added: "3.3v bus"
- note added: "MCU VI Monitor"
